Commit message: Remove wrong base rotation.

File: urdf/gp25_macro.xacro (robot description, xacro)
@@ -6,5 +6,4 @@
 		<link name="${prefix}base_link">
 			<visual>
-			        <origin rpy="0 0 3.14159"/>
 				<geometry>
 					<mesh filename="package://yaskawa_gp25_support/meshes/gp25/visual/base_axis.dae" />
@@ -15,5 +14,4 @@
 			</visual>
 			<collision>
-			        <origin rpy="0 0 3.14159"/>
 				<geometry>
 					<mesh filename="package://yaskawa_gp25_support/meshes/gp25/collision/base_axis.stl" />
@@ -43,5 +41,4 @@
 		<link name="${prefix}link_l">
 			<visual>
-				<!-- <origin rpy="1.57 3.1416 0" xyz="0 0 0"/> -->
 				<geometry>
 					<mesh filename="package://yaskawa_gp25_support/meshes/gp25/visual/l_axis.dae"/>
@@ -50,5 +47,4 @@
 			</visual>
 			<collision>
-				<!-- <origin rpy="1.57 3.1416 0" xyz="0 0 0"/> -->
 				<geometry>
 					<mesh filename="package://yaskawa_gp25_support/meshes/gp25/collision/l_axis.stl" />
@@ -59,5 +55,4 @@
 		<link name="${prefix}link_u">
 			<visual>
-				<!-- <origin rpy="1.57 -3.1415 0" xyz="0 0 0"/> -->
 				<geometry>
 					<mesh filename="package://yaskawa_gp25_support/meshes/gp25/visual/u_axis.dae"/>
@@ -66,5 +61,4 @@
 			</visual>
 			<collision>
-				<!-- <origin rpy="1.57 -3.1415 0" xyz="0 0 0"/> -->
 				<geometry>
 					<mesh filename="package://yaskawa_gp25_support/meshes/gp25/collision/u_axis.stl" />
@@ -75,5 +69,4 @@
 		<link name="${prefix}link_r">
 			<visual>
-				<!-- <origin rpy="0 0 3.1416" xyz="0 0 0"/> -->
 				<geometry>
 					<mesh filename="package://yaskawa_gp25_support/meshes/gp25/visual/r_axis.dae"/>
@@ -82,5 +75,4 @@
 			</visual>
 			<collision>
-				<!-- <origin rpy="0 0 3.1416" xyz="0 0 0"/> -->
 				<geometry>
 					<mesh filename="package://yaskawa_gp25_support/meshes/gp25/collision/r_axis.stl" />
@@ -91,5 +83,4 @@
 		<link name="${prefix}link_b">
 			<visual>
-				<!-- <origin rpy="-1.57 0 3.1416" xyz="0 0 0"/> -->
 				<geometry>
 					<mesh filename="package://yaskawa_gp25_support/meshes/gp25/visual/b_axis.dae"/>
@@ -98,5 +89,4 @@
 			</visual>
 			<collision>
-				<!-- <origin rpy="-1.57 0 3.1416" xyz="0 0 0"/> -->
 				<geometry>
 					<mesh filename="package://yaskawa_gp25_support/meshes/gp25/collision/b_axis.stl" />

Commit message: Remove identity rotations from URDF.

File: urdf/gp25_macro.xacro (robot description, xacro)
@@ -120,5 +120,5 @@
 			<parent link="${prefix}base_link"/>
 			<child link="${prefix}link_s"/>
-			<origin xyz="0 0 0" rpy="0 0 0"/>
+			<origin xyz="0 0 0" />
 			<axis xyz="0 0 1" />
 			<limit lower="${-180 / 180.0 * pi}" upper="${180 / 180.0 * pi}" effort="100" velocity="3.44" />
@@ -127,5 +127,5 @@
 			<parent link="${prefix}link_s"/>
 			<child link="${prefix}link_l"/>
-			<origin xyz="0.150 0 0.505" rpy="0 0 0"/>
+			<origin xyz="0.150 0 0.505" />
 			<axis xyz="0 1 0" />
 			<limit lower="${-105 / 180.0 * pi}" upper="${155 / 180.0 * pi}" effort="100" velocity="3.32" />
@@ -134,5 +134,5 @@
 			<parent link="${prefix}link_l"/>
 			<child link="${prefix}link_u"/>
-			<origin xyz="0 0 0.760" rpy="0 0 0"/>
+			<origin xyz="0 0 0.760" />
 			<axis xyz="0 -1 0" />
 			<!-- Limited wrt to datasheet to prevent self-collisions -->
@@ -142,5 +142,5 @@
 			<parent link="${prefix}link_u"/>
 			<child link="${prefix}link_r"/>
-			<origin xyz="0 0 0.200" rpy="0 0 0"/>
+			<origin xyz="0 0 0.200" />
 			<axis xyz="-1 0 0" />
 			<limit lower="${-200 / 180.0 * pi}" upper="${200 / 180.0 * pi}" effort="100" velocity="7.16" />
@@ -149,5 +149,5 @@
 			<parent link="${prefix}link_r"/>
 			<child link="${prefix}link_b"/>
-			<origin xyz="0.795 0 0" rpy="0 0 0"/>
+			<origin xyz="0.795 0 0" />
 			<axis xyz="0 -1 0" />
 			<limit lower="${-150 / 180.0 * pi}" upper="${150 / 180.0 * pi}" effort="100" velocity="7.16" />
@@ -156,5 +156,5 @@
 			<parent link="${prefix}link_b"/>
 			<child link="${prefix}link_t"/>
-			<origin xyz="0.100 0 0" rpy="0 0 0"/>
+			<origin xyz="0.100 0 0" />
 			<axis xyz="-1 0 0" />
 			<limit lower="${-455 / 180.0 * pi}" upper="${455 / 180.0 * pi}" effort="100" velocity="10.82" />
